File: heater.kicad_pcb (KiCad board)
At the start: 2 copper layers, 100 x 175 mm, 33 parts, among them Q1 IRFP4668PBF, Q2 IRFP4668PBF

Commit message: fix
Parts:
- added H3: 48Vin, MountingHole:MountingHole_8.4mm_M8_Pad, F.Cu at (37.0, 27.0)
- added H4: GND, MountingHole:MountingHole_8.4mm_M8_Pad, F.Cu at (117.0, 27.0)
- L1, L2: footprint Inductor_THT:L_Toroid_Vertical_L28.6mm_W14.3mm_P11.43mm_Bourns_5700 -> Inductor_THT:L_Toroid_Vertical_L31.8mm_W15.9mm_P13.50mm_Bourns_5700
- moved D3 28.2 mm to (51.0, 142.4)
- moved D4 28.2 mm to (103.0, 142.4)
- moved R2 28.2 mm to (45.0, 144.9)
- moved R9 28.2 mm to (109.0, 144.9)
- moved Q1 21.0 mm to (33.8, 146.4)
- moved Q2 21.0 mm to (120.0, 135.6)
- moved H2 17.5 mm to (117.0, 182.0)
- moved H1 16.5 mm to (37.0, 182.0)
- moved R3 3.00 mm to (120.0, 101.9)
- moved R4 2.92 mm to (34.0, 102.0)
- moved L1 0.13 mm to (104.3, 55.1)
Routing:
- net C1: track 234.8 -> 53.3 mm
- net C2: track 233.2 -> 51.8 mm
- net VCC: track 198.6 -> 127.4 mm
- net Net-(Q1-G): track 41.6 -> 14.8 mm
- net Net-(D4-K): track 61.8 -> 73.3 mm
- net Net-(D3-K): track 61.8 -> 70.4 mm
- net Net-(Q2-G): track 27.5 -> 25.6 mm

Commit message: Update heater.kicad_pcb
Other:
- board text added: "Coil"
- board text added: "GND"
- board text added: "Induction Heater Revision 1.0 Designed by: Kyle Schmerge"
- board text added: "VIN"
Changed lines of the file:
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@@
 		(layer "Edge.Cuts")
+	)
+	(gr_text "VIN"
+		(at 51 27 90)
+		(layer "F.SilkS")
+		(effects
+			(font
+				(size 6 6)
+				(thickness 0.4)
+			)
+		)
+	)
+	(gr_text "GND"
+		(at 104.75 27 90)
+		(layer "F.SilkS")
+		(effects
+			(font
+				(size 6 6)
+				(thickness 0.4)
+			)
+		)
+	)
+	(gr_text "Coil"
+		(at 76.75 182.25 0)
+		(layer "F.SilkS")
+		(effects
+			(font
+				(size 8 8)
+				(thickness 0.4)
+			)
+		)
+	)
+	(gr_text "Induction Heater Revision 1.0\nDesigned by:\nKyle Schmerge"
+		(at 79.5 89.25 90)
+		(layer "B.SilkS")
+		(effects
+			(font
+				(size 1 1)
+				(thickness 0.1)
+			)
+			(justify left bottom mirror)
+		)
 	)
 	(segment
