File: heater.kicad_sch (KiCad schematic)
At the start: 31 parts, among them Q1 IRFP4668PBF, Q2 IRFP4668PBF

Commit message: a
Parts:
- added H1: Coil 1, MountingHole:MountingHole_8.4mm_M8_Pad, symbol Mechanical:MountingHole_Pad
- added H2: Coil 2, MountingHole:MountingHole_8.4mm_M8_Pad, symbol Mechanical:MountingHole_Pad
- added HS1, HS2: Heatsink, symbol Mechanical:Heatsink
- C1, C2: Manufacturer Part Number (none) -> FG26X7S2A225KRT06; Vendor Part Number (none) -> 445-173459-1-ND
- C10, C11, C12, C3, C4, C5, C6, C7, C8, C9: footprint (none) -> Capacitor_THT:C_Rect_L31.5mm_W11.0mm_P27.50mm_MKS4; Manufacturer Part Number (none) -> MKP1J034706B00KSSD; Vendor Part Number (none) -> 1928-1437-ND
- D1: footprint (none) -> LED_THT:LED_D5.0mm; Manufacturer Part Number (none) -> WP7113ID; Vendor Part Number (none) -> 754-1264-ND
- D2: footprint (none) -> Diode_THT:D_DO-201AD_P15.24mm_Horizontal; Manufacturer Part Number (none) -> SB5H100-E3/54; Vendor Part Number (none) -> SB5H100-E3/54GICT-ND
- D5, D6: value D -> FR307; footprint (none) -> Diode_THT:D_DO-201AD_P15.24mm_Horizontal; Manufacturer Part Number (none) -> FR307G; Vendor Part Number (none) -> 1801-FR307GCT-ND
- Q1, Q2: footprint (none) -> Package_TO_SOT_THT:TO-247-3_Vertical; Manufacturer Part Number (none) -> IRFP4668PBF; Vendor Part Number (none) -> IRFP4668PBF-ND
- R1: footprint (none) -> Resistor_THT:R_Axial_DIN0207_L6.3mm_D2.5mm_P10.16mm_Horizontal; Manufacturer Part Number (none) -> CF12JT4K70; Vendor Part Number (none) -> CF12JT4K70CT-ND
- R2, R9: footprint (none) -> Resistor_THT:R_Axial_DIN0207_L6.3mm_D2.5mm_P10.16mm_Horizontal; Manufacturer Part Number (none) -> CFR-50JB-52-18R; Vendor Part Number (none) -> 13-CFR-50JB-52-18R-ND
- R3, R4: footprint (none) -> Resistor_THT:R_Axial_DIN0207_L6.3mm_D2.5mm_P10.16mm_Horizontal; Manufacturer Part Number (none) -> CF12JT10K0; Vendor Part Number (none) -> CF12JT10K0CT-ND
- R5, R8: footprint (none) -> Resistor_THT:R_Axial_DIN0918_L18.0mm_D9.0mm_P30.48mm_Horizontal; Manufacturer Part Number (none) -> ROX5SSJ470R; Vendor Part Number (none) -> A142792CT-ND
- R6, R7: footprint (none) -> Resistor_THT:R_Axial_DIN0918_L18.0mm_D9.0mm_P30.48mm_Horizontal; Manufacturer Part Number (none) -> ROX5SSJ47R; Vendor Part Number (none) -> A142768CT-ND
Connections:
- net C1: now also D6.1 (K), H1.1; no longer D5.1 (K)
- net C2: now also D5.1 (K), H2.1; no longer D6.1 (K)
Other:
- moved on the sheet: D5, D6

Commit message: fix
Parts:
- added H3: 48Vin, MountingHole:MountingHole_8.4mm_M8_Pad, symbol Mechanical:MountingHole_Pad
- added H4: GND, MountingHole:MountingHole_8.4mm_M8_Pad, symbol Mechanical:MountingHole_Pad
- L1, L2: footprint Inductor_THT:L_Toroid_Vertical_L28.6mm_W14.3mm_P11.43mm_Bourns_5700 -> Inductor_THT:L_Toroid_Vertical_L31.8mm_W15.9mm_P13.50mm_Bourns_5700; Manufacturer Part Number (none) -> 2312-V-RC; Vendor Part Number (none) -> M8888-ND
Connections:
- net GND: now also H4.1
- net VCC: now also H3.1

Commit message: fix mosfet part No.
Parts:
- Q1, Q2: Manufacturer Part Number IRFP4668PBF -> IRFP4668PBFXKMA1; Vendor Part Number IRFP4668PBF-ND -> 448-IRFP4668PBFXKMA1-ND
Changed lines of the file:
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@@
 			)
 		)
-		(property "Manufacturer Part Number" "IRFP4668PBF"
+		(property "Manufacturer Part Number" "IRFP4668PBFXKMA1"
 			(at 82.55 120.65 0)
 			(effects
@@
 			)
 		)
-		(property "Vendor Part Number" "IRFP4668PBF-ND"
+		(property "Vendor Part Number" "448-IRFP4668PBFXKMA1-ND"
 			(at 82.55 120.65 0)
 			(effects
@@
 			)
 		)
-		(property "Manufacturer Part Number" "IRFP4668PBF"
+		(property "Manufacturer Part Number" "IRFP4668PBFXKMA1"
 			(at 120.65 120.65 0)
 			(effects
@@
 			)
 		)
-		(property "Vendor Part Number" "IRFP4668PBF-ND"
+		(property "Vendor Part Number" "448-IRFP4668PBFXKMA1-ND"
 			(at 120.65 120.65 0)
 			(effects
