File: v2/heater.kicad_pcb (KiCad board)
At the start: 2 copper layers, 100 x 175 mm, 35 parts, among them Q1 IRFP4668PBF, Q2 IRFP4668PBF

Commit message: work on v2
Parts:
- added C13: 470nF, Capacitor_THT:C_Rect_L31.5mm_W11.0mm_P27.50mm_MKS4, F.Cu at (171.2, 244.0)
- added C14: 470nF, Capacitor_THT:C_Rect_L31.5mm_W11.0mm_P27.50mm_MKS4, F.Cu at (171.2, 256.0)
- added C15: 470nF, Capacitor_THT:C_Rect_L31.5mm_W11.0mm_P27.50mm_MKS4, F.Cu at (171.2, 268.0)
- added C16: 470nF, Capacitor_THT:C_Rect_L31.5mm_W11.0mm_P27.50mm_MKS4, F.Cu at (171.2, 280.0)
- added C17: 100μF, Capacitor_THT:C_Radial_D10.0mm_H20.0mm_P5.00mm, F.Cu at (161.0, 37.8)
- added C18: 330μF, Capacitor_THT:C_Radial_D12.5mm_H25.0mm_P5.00mm, F.Cu at (161.0, 51.5)
- added D7: LED, LED_THT:LED_D5.0mm, F.Cu at (205.0, 60.0)
- added D8: LED, LED_THT:LED_D5.0mm, F.Cu at (205.0, 67.5)
- added D9: 1N5819, Diode_THT:D_DO-41_SOD81_P10.16mm_Horizontal, F.Cu at (173.4, 49.2)
- added H5: MountingHole_Pad, MountingHole:MountingHole_5.3mm_M5_DIN965_Pad, F.Cu at (130.0, 75.0)
- added H6: MountingHole_Pad, MountingHole:MountingHole_5.3mm_M5_DIN965_Pad, F.Cu at (240.0, 75.0)
- added H7: MountingHole_Pad, MountingHole:MountingHole_5.3mm_M5_DIN965_Pad, F.Cu at (150.0, 265.0)
- added H8: MountingHole_Pad, MountingHole:MountingHole_5.3mm_M5_DIN965_Pad, F.Cu at (220.0, 265.0)
- added HS1: Heatsink, footprints:694-50, F.Cu at (129.3, 248.0)
- added HS2: Heatsink, footprints:694-50, F.Cu at (129.3, 194.0)
- added HS3: Heatsink, footprints:694-50, F.Cu at (129.3, 140.0)
- added HS4: Heatsink, footprints:694-50, F.Cu at (240.7, 140.0)
- added HS5: Heatsink, footprints:694-50, F.Cu at (240.7, 194.0)
- added HS6: Heatsink, footprints:694-50, F.Cu at (240.7, 248.0)
- added L3: 330μH, footprints:WE-PD_1210, F.Cu at (192.0, 44.7)
- added M1: Fan_4pin, Connector_Molex:Molex_KK-254_AE-6410-04A_1x04_P2.54mm_Vertical, F.Cu at (205.0, 41.0)
- added M2: Fan_4pin, Connector_Molex:Molex_KK-254_AE-6410-04A_1x04_P2.54mm_Vertical, F.Cu at (205.0, 54.0)
- added Q1: IRFP4668PBF, Package_TO_SOT_THT:TO-247-3_Vertical, F.Cu at (135.0, 253.4)
- added Q2: IRFP4668PBF, Package_TO_SOT_THT:TO-247-3_Vertical, F.Cu at (135.0, 199.4)
- added Q5: IRFP4668PBF, Package_TO_SOT_THT:TO-247-3_Vertical, F.Cu at (235.0, 188.6)
- added Q6: IRFP4668PBF, Package_TO_SOT_THT:TO-247-3_Vertical, F.Cu at (235.0, 242.6)
- added R10: 18Ω, Resistor_THT:R_Axial_DIN0207_L6.3mm_D2.5mm_P10.16mm_Horizontal, F.Cu at (143.0, 188.9)
- added R11: 18Ω, Resistor_THT:R_Axial_DIN0207_L6.3mm_D2.5mm_P10.16mm_Horizontal, F.Cu at (143.0, 242.9)
- added R12: 18Ω, Resistor_THT:R_Axial_DIN0207_L6.3mm_D2.5mm_P10.16mm_Horizontal, F.Cu at (227.0, 253.1)
- added R13: 18Ω, Resistor_THT:R_Axial_DIN0207_L6.3mm_D2.5mm_P10.16mm_Horizontal, F.Cu at (227.0, 199.1)
- added R14: 6.8kΩ, Resistor_SMD:R_1206_3216Metric_Pad1.30x1.75mm_HandSolder, F.Cu at (216.0, 35.0)
- added R15: 4.7kΩ, Resistor_SMD:R_1206_3216Metric_Pad1.30x1.75mm_HandSolder, F.Cu at (221.0, 35.0)
- added R16: 820Ω, Resistor_SMD:R_1206_3216Metric_Pad1.30x1.75mm_HandSolder, F.Cu at (200.0, 60.0)
- added R17: 6.8kΩ, Resistor_SMD:R_1206_3216Metric_Pad1.30x1.75mm_HandSolder, F.Cu at (216.0, 39.0)
- added R18: 4.7kΩ, Resistor_SMD:R_1206_3216Metric_Pad1.30x1.75mm_HandSolder, F.Cu at (221.0, 39.0)
- added R19: 820Ω, Resistor_SMD:R_1206_3216Metric_Pad1.30x1.75mm_HandSolder, F.Cu at (200.0, 64.0)
- added U1: LM2575-12BU, Package_TO_SOT_SMD:TO-263-5_TabPin3, F.Cu at (178.5, 36.8)
- L1, L2: value 100μH -> 70μH
- R5, R8: value 470Ω -> 1kΩ
- R6, R7: value 47Ω -> 150Ω
- moved H1 152.7 mm to (145.0, 290.0)
- moved H2 152.7 mm to (225.0, 290.0)
- moved D5 142.2 mm to (150.0, 172.6)
- moved D6 140.5 mm to (220.0, 172.4)
- moved C1 135.7 mm to (150.0, 155.2)
- moved C3 133.2 mm to (171.2, 124.0)
- moved C4 132.9 mm to (171.2, 136.0)
- moved C5 132.6 mm to (171.2, 148.0)
- moved C6 132.3 mm to (171.2, 160.0)
- moved C7 131.9 mm to (171.2, 172.0)
- moved C8 131.6 mm to (171.2, 184.0)
- moved C9 131.3 mm to (171.2, 196.0)
- moved C10 131.0 mm to (171.2, 208.0)
- moved C11 130.7 mm to (171.2, 220.0)
- moved C12 130.4 mm to (171.2, 232.0)
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- renumbered Q1 to Q3, Q2 to Q4
Routing:
- net +12V: track 0.00 -> 106.1 mm
- net Net-(D4-K): track 73.3 -> 148.3 mm
- net Net-(D3-K): track 70.4 -> 144.9 mm
- net GND: track 0.00 -> 39.6 mm, vias 0 -> 3
- net Net-(D9-K): track 0.00 -> 28.2 mm, vias 0 -> 1
- net Net-(D7-K): track 0.00 -> 25.7 mm
- net Net-(C2-Pad1): track 38.8 -> 14.7 mm
- net Net-(C1-Pad1): track 38.2 -> 14.6 mm
- net Net-(D8-K): track 0.00 -> 22.0 mm
- net Net-(M2-PWM): track 0.00 -> 17.5 mm
- net Net-(Q4-G): track 25.6 -> 8.15 mm
- net Net-(M1-PWM): track 0.00 -> 15.1 mm
- net Net-(D8-A): track 0.00 -> 11.0 mm
- net Net-(Q6-G): track 0.00 -> 8.15 mm
- net Net-(Q5-G): track 0.00 -> 8.15 mm
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- added copper zone on B.Cu, net C1
- added copper zone on B.Cu, net C2
- added copper zone on B.Cu, net VCC
- removed copper zone on F.Cu, net GND
Other:
- board size 100 x 175 mm -> 130 x 280 mm
- board text added: "Fan1"
- board text added: "Fan2"
- board text added: "Induction Heater Revision 2.0 Designed by: Kyle Schmerge"
- board text added: "Power"
- board text removed: "Induction Heater Revision 1.0 Designed by: Kyle Schmerge"

Commit message: w
Parts:
- added H10: MP, MountingHole:MountingHole_3.2mm_M3_DIN965_Pad, F.Cu at (164.0, 95.0)
- added H11: MP, MountingHole:MountingHole_3.2mm_M3_DIN965_Pad, F.Cu at (164.0, 85.0)
- added H12: MP, MountingHole:MountingHole_3.2mm_M3_DIN965_Pad, F.Cu at (211.0, 279.0)
- added H13: MP, MountingHole:MountingHole_3.2mm_M3_DIN965_Pad, F.Cu at (206.0, 95.0)
- added H14: MP, MountingHole:MountingHole_3.2mm_M3_DIN965_Pad, F.Cu at (206.0, 85.0)
- added H15: MP, MountingHole:MountingHole_3.2mm_M3_DIN965_Pad, F.Cu at (125.0, 51.5)
- added H16: MP, MountingHole:MountingHole_3.2mm_M3_DIN965_Pad, F.Cu at (125.0, 66.0)
- added H17: MP, MountingHole:MountingHole_3.2mm_M3_DIN965_Pad, F.Cu at (245.0, 66.0)
- added H9: MP, MountingHole:MountingHole_3.2mm_M3_DIN965_Pad, F.Cu at (162.5, 279.0)
- C10, C11, C12, C13, C14, C15, C16, C3, C4, C5, C6, C7, C8, C9: value 470nF -> 330nF; footprint Capacitor_THT:C_Rect_L31.5mm_W11.0mm_P27.50mm_MKS4 -> Capacitor_THT:C_Rect_L31.5mm_W15.0mm_P27.50mm_MKS4
- L1, L2: footprint Inductor_THT:L_Toroid_Vertical_L31.8mm_W15.9mm_P13.50mm_Bourns_5700 -> footprints:L_Toroid_Vertical_L39.9mm_W32.4mm_P30.0mm
- moved C3 38.0 mm to (171.2, 86.0)
- moved H5 35.0 mm to (130.0, 40.0)
- moved H6 35.0 mm to (240.0, 40.0)
- moved C4 34.0 mm to (171.2, 102.0)
- moved D8 30.7 mm to (213.7, 38.0)
- moved C5 30.0 mm to (171.2, 118.0)
- moved M2 27.8 mm to (219.0, 30.0), turned to 180 degrees
- moved R14 27.7 mm to (189.0, 29.0)
- moved R15 27.7 mm to (194.0, 29.0)
- moved R17 27.7 mm to (189.0, 33.0)
- moved R18 27.7 mm to (194.0, 33.0)
- moved C6 26.0 mm to (171.2, 134.0)
- moved R19 25.0 mm to (215.0, 44.0)
- moved D7 22.2 mm to (201.7, 38.0)
- moved C7 22.0 mm to (171.2, 150.0)
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Routing:
- net VCC: track 119.5 -> 173.8 mm
- net Net-(D7-K): track 25.7 -> 8.08 mm
- net +12V: track 106.1 -> 121.1 mm
- net Net-(D8-K): track 22.0 -> 8.08 mm
- net Net-(M2-PWM): track 17.5 -> 25.4 mm, vias 0 -> 1
- net Net-(D8-A): track 11.0 -> 6.12 mm
- net Net-(M1-PWM): track 15.1 -> 10.5 mm
- net GND: track 39.6 -> 36.7 mm, vias 3 -> 1
- net C1: track 51.9 -> 54.0 mm
- net Net-(D7-A): track 7.70 -> 6.12 mm
- net C2: track 52.3 -> 51.5 mm
- added copper zone on F.Cu, net GND
