File: v2/heater.kicad_pcb (KiCad board)
At the start: 2 copper layers, 130 x 280 mm, 81 parts, among them M1 Fan_4pin, M2 Fan_4pin, Q1 IRFP4668PBF, Q2 IRFP4668PBF, Q3 IRFP4668PBF, Q4 IRFP4668PBF, Q5 IRFP4668PBF, Q6 IRFP4668PBF, U1 LM2575-12BU

Commit message: fixes
Parts:
- moved D7 93.9 mm to (286.7, 78.0)
- moved D8 93.9 mm to (298.7, 78.0)
- moved D9 93.9 mm to (258.4, 89.2)
- moved U1 93.9 mm to (263.5, 76.8)
- moved R11 93.9 mm to (228.0, 282.9)
- moved C1 93.9 mm to (235.0, 195.2)
- moved C10 93.9 mm to (256.2, 238.0)
- moved C11 93.9 mm to (256.2, 254.0)
- moved C12 93.9 mm to (256.2, 270.0)
- moved C13 93.9 mm to (256.2, 286.0)
- moved C14 93.9 mm to (256.2, 302.0)
- moved C15 93.9 mm to (256.2, 318.0)
- moved C16 93.9 mm to (256.2, 334.0)
- moved C17 93.9 mm to (246.0, 77.8)
- moved C18 93.9 mm to (246.0, 91.5)
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Routing:
- net GND: vias 1 -> 87

Commit message: final touches
Routing:
- net VCC: track 173.8 -> 175.2 mm
Other:
- outline, holes or cut-outs redrawn
- board text removed: "Coil"
