File: v2/fan_control.kicad_sch (KiCad schematic)
At the start: 15 parts, among them M1 Fan_4pin, M2 Fan_4pin, U1 LM2575-12BU

Commit message: work on v2
Parts:
- added H5, H6, H7, H8: MountingHole_Pad, MountingHole:MountingHole_5.3mm_M5_DIN965_Pad, symbol Mechanical:MountingHole_Pad
- C17: footprint Capacitor_THT:C_Rect_L31.5mm_W11.0mm_P27.50mm_MKS4 -> Capacitor_THT:C_Radial_D10.0mm_H20.0mm_P5.00mm; Manufacturer Part Number (none) -> 100ZLH100MEFC10X20; Vendor Part Number (none) -> 1189-1887-ND
- C18: footprint Capacitor_THT:C_Rect_L31.5mm_W11.0mm_P27.50mm_MKS4 -> Capacitor_THT:C_Radial_D12.5mm_H25.0mm_P5.00mm; Manufacturer Part Number (none) -> UVZ2A331MHD1TO; Vendor Part Number (none) -> 493-13506-1-ND
- D9: Manufacturer Part Number (none) -> 1N5819; Vendor (none) -> Digi-Key; Vendor Part Number (none) -> 497-6610-1-ND
- L3: footprint (none) -> footprints:WE-PD_1210; Manufacturer Part Number (none) -> 7447709331; Vendor (none) -> Digi-Key; Vendor Part Number (none) -> 732-1698-1-ND
- M1, M2: footprint (none) -> Connector_Molex:Molex_KK-254_AE-6410-04A_1x04_P2.54mm_Vertical; Manufacturer Part Number (none) -> 0022292041; Vendor (none) -> Digi-Key; Vendor Part Number (none) -> WM2746-ND
- R14, R15, R16, R17, R18, R19: footprint (none) -> Resistor_SMD:R_1206_3216Metric_Pad1.30x1.75mm_HandSolder; Vendor (none) -> Digi-Key
- U1: Manufacturer Part Number (none) -> LM2575HVS-12/NOPB; Vendor (none) -> Digi-Key; Vendor Part Number (none) -> LM2575HVS-12/NOPB-ND
Connections:
- no-connect marks 0 -> 4

Commit message: final touches
Parts:
- R14, R17: Manufacturer Part Number (none) -> RC1206FR-076K8L; Vendor Part Number (none) -> 311-6.80KFRCT-ND
- R15, R18: Manufacturer Part Number (none) -> RC1206FR-074K7L; Vendor Part Number (none) -> 311-4.70KFRCT-ND
- R16, R19: Manufacturer Part Number (none) -> CRGCQ1206F820R; Vendor Part Number (none) -> A129809CT-ND
Changed lines of the file:
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@@
+			)
+		)
+		(property "Manufacturer Part Number" "CRGCQ1206F820R"
+			(at 105.41 43.18 0)
+			(hide yes)
+			(show_name no)
+			(do_not_autoplace no)
+			(effects
+				(font
+					(size 1.27 1.27)
+				)
+			)
+		)
+		(property "Vendor Part Number" "A129809CT-ND"
+			(at 105.41 43.18 0)
+			(hide yes)
+			(show_name no)
+			(do_not_autoplace no)
+			(effects
+				(font
+					(size 1.27 1.27)
+				)
 			)
 		)
@@
 		)
 		(property "Vendor" "Digi-Key"
+			(at 105.41 104.14 0)
+			(hide yes)
+			(show_name no)
+			(do_not_autoplace no)
+			(effects
+				(font
+					(size 1.27 1.27)
+				)
+			)
+		)
+		(property "Manufacturer Part Number" "CRGCQ1206F820R"
+			(at 105.41 104.14 0)
+			(hide yes)
+			(show_name no)
+			(do_not_autoplace no)
+			(effects
+				(font
+					(size 1.27 1.27)
+				)
+			)
+		)
+		(property "Vendor Part Number" "A129809CT-ND"
 			(at 105.41 104.14 0)
 			(hide yes)
@@
 			)
 		)
+		(property "Manufacturer Part Number" "RC1206FR-074K7L"
+			(at 85.09 71.12 0)
+			(hide yes)
+			(show_name no)
+			(do_not_autoplace no)
+			(effects
+				(font
+					(size 1.27 1.27)
+				)
+			)
+		)
+		(property "Vendor Part Number" "311-4.70KFRCT-ND"
+			(at 85.09 71.12 0)
+			(hide yes)
+			(show_name no)
+			(do_not_autoplace no)
+			(effects
+				(font
+					(size 1.27 1.27)
+				)
+			)
+		)
 		(pin "1"
 		)
@@
 			)
 		)
+		(property "Manufacturer Part Number" "RC1206FR-076K8L"
+			(at 85.09 58.42 0)
+			(hide yes)
+			(show_name no)
+			(do_not_autoplace no)
+			(effects
+				(font
+					(size 1.27 1.27)
+				)
+			)
+		)
+		(property "Vendor Part Number" "311-6.80KFRCT-ND"
+			(at 85.09 58.42 0)
+			(hide yes)
+			(show_name no)
+			(do_not_autoplace no)
+			(effects
+				(font
+					(size 1.27 1.27)
+				)
+			)
+		)
 		(pin "1"
 		)
@@
 			)
 		)
+		(property "Manufacturer Part Number" "RC1206FR-074K7L"
+			(at 85.09 132.08 0)
+			(hide yes)
+			(show_name no)
+			(do_not_autoplace no)
+			(effects
+				(font
+					(size 1.27 1.27)
+				)
+			)
+		)
+		(property "Vendor Part Number" "311-4.70KFRCT-ND"
+			(at 85.09 132.08 0)
+			(hide yes)
+			(show_name no)
+			(do_not_autoplace no)
+			(effects
+				(font
+					(size 1.27 1.27)
+				)
+			)
+		)
 		(pin "1"
 		)
@@
 			(at 85.09 119.38 0)
 			(hide yes)
+			(show_name no)
+			(do_not_autoplace no)
+			(effects
+				(font
+					(size 1.27 1.27)
+				)
+			)
+		)
+		(property "Manufacturer Part Number" "RC1206FR-076K8L"
+			(at 85.09 119.38 0)
+			(hide yes)
+			(show_name no)
+			(do_not_autoplace no)
+			(effects
+				(font
+					(size 1.27 1.27)
+				)
+			)
+		)
+		(property "Vendor Part Number" "311-6.80KFRCT-ND"
+			(at 85.09 119.38 0)
+			(hide yes)
