File: v2/heater.kicad_sch (KiCad schematic)
At the start: 53 parts, among them Q1 IRFP4668PBF, Q2 IRFP4668PBF, Q3 IRFP4668PBF, Q4 IRFP4668PBF, Q5 IRFP4668PBF, Q6 IRFP4668PBF

Commit message: work on v2
Parts:
- HS1, HS2, HS3, HS4, HS5, HS6: footprint (none) -> footprints:694-50
- L1, L2: Manufacturer Part Number 2312-V-RC -> (none); Vendor Part Number M8888-ND -> (none)
- R5, R8: value 470Ω -> 1kΩ; Manufacturer Part Number ROX5SSJ470R -> (none); Vendor Part Number A142792CT-ND -> (none)
- R6, R7: value 47Ω -> 150Ω; Manufacturer Part Number ROX5SSJ47R -> (none); Vendor Part Number A142768CT-ND -> (none)
Other:
- moved on the sheet: C10, C11, C12, C13, C14, C15, C16, C3, C4, C5, C6, C7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

Commit message: w
Parts:
- added H10, H11, H12, H13, H14, H15, H16, H17, H9: MP, MountingHole:MountingHole_3.2mm_M3_DIN965_Pad, symbol Mechanical:MountingHole_Pad
- C10, C11, C12, C13, C14, C15, C16, C3, C4, C5, C6, C7, C8, C9: value 470nF -> 330nF; footprint Capacitor_THT:C_Rect_L31.5mm_W11.0mm_P27.50mm_MKS4 -> Capacitor_THT:C_Rect_L31.5mm_W15.0mm_P27.50mm_MKS4; Manufacturer Part Number MKP1J034706B00KSSD -> MKP1O133306F00KSSD; Vendor Part Number 1928-1437-ND -> 1928-1444-ND
- L1, L2: footprint Inductor_THT:L_Toroid_Vertical_L31.8mm_W15.9mm_P13.50mm_Bourns_5700 -> footprints:L_Toroid_Vertical_L39.9mm_W32.4mm_P30.0mm
Connections:
- net C1: now also H10.1, H11.1, H9.1
- net C2: now also H12.1, H13.1, H14.1
- net VCC: now also H15.1, H16.1, H17.1

Commit message: final touches
Parts:
- L1, L2: Vendor Digi-Key -> (none)
- R5, R8: Manufacturer Part Number (none) -> WS5M1001J; Vendor Part Number (none) -> WS5M1001JCT-ND
- R6, R7: Manufacturer Part Number (none) -> EP5WS150RJ; Vendor Part Number (none) -> A131370CT-ND
Changed lines of the file:
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@@
 			)
 		)
-		(property "Manufacturer Part Number" ""
+		(property "Manufacturer Part Number" "EP5WS150RJ"
 			(at 179.07 73.66 0)
 			(hide yes)
@@
 			)
 		)
-		(property "Vendor Part Number" ""
+		(property "Vendor Part Number" "A131370CT-ND"
 			(at 179.07 73.66 0)
 			(hide yes)
@@
 			)
 		)
-		(property "Vendor" "Digi-Key"
+		(property "Vendor" ""
 			(at 166.37 80.01 0)
 			(hide yes)
@@
 			)
 		)
-		(property "Manufacturer Part Number" ""
+		(property "Manufacturer Part Number" "WS5M1001J"
 			(at 179.07 87.63 0)
 			(hide yes)
@@
 			)
 		)
-		(property "Vendor Part Number" ""
+		(property "Vendor Part Number" "WS5M1001JCT-ND"
 			(at 179.07 87.63 0)
 			(hide yes)
@@
 			)
 		)
-		(property "Manufacturer Part Number" ""
+		(property "Manufacturer Part Number" "EP5WS150RJ"
 			(at 120.65 73.66 0)
 			(hide yes)
@@
 			)
 		)
-		(property "Vendor Part Number" ""
+		(property "Vendor Part Number" "A131370CT-ND"
 			(at 120.65 73.66 0)
 			(hide yes)
@@
 			)
 		)
-		(property "Vendor" "Digi-Key"
+		(property "Vendor" ""
 			(at 133.35 80.01 0)
 			(hide yes)
@@
 			)
 		)
-		(property "Manufacturer Part Number" ""
+		(property "Manufacturer Part Number" "WS5M1001J"
 			(at 120.65 87.63 0)
 			(hide yes)
@@
 			)
 		)
-		(property "Vendor Part Number" ""
+		(property "Vendor Part Number" "WS5M1001JCT-ND"
 			(at 120.65 87.63 0)
 			(hide yes)
