File: v2/heater.kicad_sch (KiCad schematic)
At the start: 62 parts, among them Q1 IRFP4668PBF, Q2 IRFP4668PBF, Q3 IRFP4668PBF, Q4 IRFP4668PBF, Q5 IRFP4668PBF, Q6 IRFP4668PBF

Commit message: w
Parts:
- removed C1, C2: 2.2μF, Capacitor_THT:C_Disc_D4.3mm_W1.9mm_P5.00mm, symbol Device:C
- removed D3, D4: 12V, Diode_THT:D_DO-15_P15.24mm_Horizontal, symbol Device:D_Zener
- removed D5, D6: FR307, Diode_THT:D_DO-201AD_P15.24mm_Horizontal, symbol Device:D
- removed HS1, HS2, HS3, HS4, HS5, HS6: Heatsink, footprints:694-50, symbol Mechanical:Heatsink
- removed Q1, Q2, Q3, Q4, Q5, Q6: IRFP4668PBF, Package_TO_SOT_THT:TO-247-3_Vertical, symbol Transistor_FET:Q_NMOS_GDS
- removed R10, R11, R12, R13, R2, R9: 18Ω, Resistor_THT:R_Axial_DIN0207_L6.3mm_D2.5mm_P10.16mm_Horizontal, symbol Device:R_US
- removed R3, R4: 10kΩ, Resistor_THT:R_Axial_DIN0207_L6.3mm_D2.5mm_P10.16mm_Horizontal, symbol Device:R_US
- removed R5, R8: 1kΩ, Resistor_THT:R_Axial_DIN0918_L18.0mm_D9.0mm_P30.48mm_Horizontal, symbol Device:R_US
- removed R6, R7: 150Ω, Resistor_THT:R_Axial_DIN0918_L18.0mm_D9.0mm_P30.48mm_Horizontal, symbol Device:R_US
Other:
- moved on the sheet: C10, C11, C12, C13, C14, C15, C16, C3, C4, C5, C6, C7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
