File: v2/pll_gate_drive.kicad_sch (KiCad schematic)
At the start: 2 parts, among them U2 4046, U3 UCC27511ADBV

Commit message: w
Parts:
- added C1: 2nF, symbol Device:C
- added C19, C20, C21, C22, C23, C24, C25: 100nF, symbol Device:C
- added C2: 10nF, symbol Device:C
- added D3, D4: 1N4148, Diode_THT:D_DO-35_SOD27_P7.62mm_Horizontal, symbol Diode:1N4148
- added HS1, HS2, HS3, HS4, HS5, HS6: Heatsink, footprints:694-50, symbol Mechanical:Heatsink
- added Q1, Q2, Q3, Q4, Q5, Q6: IRFP4668PBF, Package_TO_SOT_THT:TO-247-3_Vertical, symbol Transistor_FET:Q_NMOS_GDS
- added R10, R11, R12, R13, R2, R9: 18Ω, Resistor_THT:R_Axial_DIN0207_L6.3mm_D2.5mm_P10.16mm_Horizontal, symbol Device:R_US
- added R20: 180kΩ, Resistor_SMD:R_1206_3216Metric_Pad1.30x1.75mm_HandSolder, symbol Device:R_US
- added R3: 51kΩ, symbol Device:R_US
- added R4: 220kΩ, symbol Device:R_US
- added R5: 1kΩ, symbol Device:R_US
- added U4, U5, U6, U7, U8: UCC27511ADBV, Package_TO_SOT_SMD:SOT-23-6, symbol Driver_FET:UCC27511ADBV
- U2: value 4046 -> CD74HC4046; Manufacturer Part Number (none) -> 296-9208-5-ND; Vendor (none) -> Digi-Key; Vendor Part Number (none) -> CD74HC4046AE
Connections:
- net +12V: now also C19.1, C20.1, C21.1, C22.1, C23.1, C24.1, U4.1 (V_{DD}), U5.1 (V_{DD}), U6.1 (V_{DD}), U6.6 (IN+), U7.1 (V_{DD}), U7.6 (IN+), U8.1 (V_{DD}), U8.6 (IN+)
- net +5V: now also C25.1, D3.1 (K)
- net GND: now also U2.5 (Inh), C19.2, C2.2, C20.2, C21.2, C22.2, C23.2, C24.2, C25.2, D4.2 (A), Q1.3 (S), Q2.3 (S), Q3.3 (S), Q4.3 (S), Q5.3 (S), Q6.3 (S), R3.1, R4.1, U4.4 (GND), U4.5 (IN-), U5.4 (GND), U5.5 (IN-), U6.4 (GND), U7.4 (GND), U8.4 (GND)
- net at U3.2 (OUTH): now also U3.3 (OUTL), R2.1
- net GATE_PWM: now reaches U3.6 (IN+)
- net GATE_PWM: now also U2.3 (RefIn), U2.4 (FOUT), U4.6 (IN+), U5.6 (IN+), U6.5 (IN-), U7.5 (IN-), U8.5 (IN-)
- net at U2.11 (R1): now also R3.2
- net at U2.12 (R2): now also R4.2
- net at U2.13 (PC2): now also R5.1
- net at U2.14 (SigIn): now also D3.2 (A), D4.1 (K), R20.2
- net at U2.6 (C1): now also C1.1
- net at U2.7 (C2): now also C1.2
- net at U2.9 (VCOin): now also C2.1, R5.2
- new net: R10.1, U4.2 (OUTH), U4.3 (OUTL)
- new net: Q2.1 (G), R10.2
- new net: Q3.1 (G), R2.2
- new net: Q5.1 (G), R13.2
- new net: R12.2, U6.2 (OUTH), U6.3 (OUTL)
- new net: Q4.1 (G), R9.2
- new net: R9.1, U8.2 (OUTH), U8.3 (OUTL)
- new net: Q1.1 (G), R11.2
- new net: R13.1, U7.2 (OUTH), U7.3 (OUTL)
- new net: R11.1, U5.2 (OUTH), U5.3 (OUTL)
- new net: Q6.1 (G), R12.1
- new net C1: Q1.2 (D), Q2.2 (D), Q3.2 (D)
- new net C2: Q4.2 (D), Q5.2 (D), Q6.2 (D), R20.1
- no-connect marks 0 -> 4
Other:
- moved on the sheet: U3
