File: v2/1.0/heater.kicad_sch (KiCad schematic)
At the start: 62 parts, among them Q1 IRFP4668PBF, Q2 IRFP4668PBF, Q3 IRFP4668PBF, Q4 IRFP4668PBF, Q5 IRFP4668PBF, Q6 IRFP4668PBF

Commit message: archive and update
Other:
- removed sheet PLL & Gate Drive
- moved on the sheet: C1, C10, C11, C12, C13, C14, C15, C16, C2, C3, C4, C5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
